Commit message: Make new URDF compatible with gazebo

File: urdf/ur5_ft_grip_table_gazebo.xacro (robot description, xacro)
@@ -7,10 +7,11 @@
         <origin xyz="0 0 0" rpy="0 0 0"/>
     </xacro:robotiq_ft300>
-    <!-- Robotiq gripper -->
-    <xacro:include filename="$(find robotiq_2f_85_gripper_visualization)/urdf/robotiq_arg2f_85_model_macro.xacro" />
-    <xacro:robotiq_arg2f_85 prefix=""/>
+    <!-- Simple gripper -->
+    <xacro:include filename="$(find robot_control)/urdf/simple_gripper.xacro" />
+    <xacro:simple_gripper />
     <joint name="gripper_fix" type="fixed">
         <parent link="robotiq_ft_frame_id" />
-        <child link="robotiq_arg2f_base_link" />
+        <child link="pusher" />
+        <origin xyz="0.0 0.0 0.0" rpy="0.0 ${-pi/2} 0.0" />
     </joint>
     <!-- Table representing the boundary of the workspace -->
