Commit message: Fix URDFs for use with actual robot

File: urdf/simple_gripper.xacro (robot description, xacro)
@@ -2,7 +2,7 @@
   <robot xmlns:xacro="http://www.ros.org/wiki/xacro" name="simple_gripper">
   <xacro:macro name="simple_gripper">
-    <!-- <material name="black">
-      <color rgba="0 0 0.8 1"/>
-    </material> -->
+    <material name="grey">
+      <color rgba="0.7 0.7 0.7 1"/>
+    </material>
     <link name="pusher">
       <visual>
@@ -10,5 +10,5 @@
           <cylinder length="0.085" radius="0.0375"/>
         </geometry>
-        <material name="black"/>
+        <material name="grey"/>
         <origin rpy="0 1.57075 0" xyz="0.04625 0 0"/>
       </visual>
@@ -29,5 +29,5 @@
           <box size="0.11 0.025 0.02"/>
         </geometry>
-        <material name="black"/>
+        <material name="grey"/>
         <origin rpy="0 0 0" xyz="0.055 0.025 0"/>
       </visual>
@@ -53,5 +53,5 @@
           <box size="0.11 0.025 0.02"/>
         </geometry>
-        <material name="black"/>
+        <material name="grey"/>
         <origin rpy="0 0 0" xyz="0.055 -0.025 0"/>
       </visual>

File: urdf/table.xacro (robot description, xacro)
@@ -1,4 +1,7 @@
 <?xml version="1.0"?>
   <robot xmlns:xacro="http://www.ros.org/wiki/xacro" name="table">
+    <material name="blue">
+      <color rgba="0 0 0.8 1"/>
+    </material>
     <xacro:macro name="table">
       <link name="table_base">
@@ -7,4 +10,5 @@
             <box size="4.0 4.0 0.01"/>
           </geometry>
+          <material name="blue"/>
         </visual>
         <collision>

File: urdf/ur5_ft_grip_table.xacro (robot description, xacro)
@@ -16,5 +16,5 @@
     <!-- Table representing the boundary of the workspace -->
     <xacro:include filename="$(find robot_control)/urdf/table.xacro" />
-    <!-- <xacro:table /> -->
+    <xacro:table />
     <!-- UR5 robot (parameters should be defined in launch files)-->
     <xacro:include filename="$(find ur_description)/urdf/inc/ur_macro.xacro" />
